File: theyseemerolling-bldc.kicad_pcb (KiCad board)
At the start: 2 copper layers, 204 parts, among them J1 Conn_Debug, Q1 BSS138, Q10 NMOS-T252, Q11 NMOS-T252, Q12 BSS138, Q13 BSS138, Q14 NMOS-T252, Q15 NMOS-T252, Q16 BSS138, Q17 BSS138, Q18 NMOS-T252, Q19 NMOS-T252, Q2 BSS138, Q20 BSS138, Q21 BSS138, Q22 BSS138, Q23 BSS138, Q24 BSS138, Q25 BSS138, Q26 BSS138, Q27 BSS138, Q28 BSS138, Q29 NMOS-T252, Q3 BSS138, Q30 NMOS-T252, Q31 BSS138, Q32 BSS138, Q33 NMOS-T252, Q34 NMOS-T252, Q35 BSS138, Q36 BSS138, Q37 NMOS-T252, Q38 NMOS-T252, Q4 BSS138, Q5 BSS138, Q6 BSS138, Q7 BSS138, Q8 BSS138, Q9 BSS138, U1 STM32F405RGTx, U10 LMC555xM, U11 L6388E, U12 L6388E, U13 L6388E, U14 SN74LVC1G32, U15 ACS711xLCTR-12AB, U16 SN74LVC1G32, U17 LM358, U18 LMC555xM, U19 L6388E, U20 L6388E, U21 L6388E, U3 LM358, U4 LM317L_SO8, U5 TCAN332, U6 LD1117S50TR_SOT223, U7 LD1117S33TR_SOT223, U8 ACS711xLCTR-12AB, U9 LM358, Y1 8Mhz

Commit message: Fix schematics, route
Parts:
- removed the Q18 at (251.0, 118.0)
- added C27: 100n, Capacitor_SMD:C_0805_2012Metric_Pad1.15x1.40mm_HandSolder, F.Cu at (206.2, 83.5)
- added Q19: NMOS-T252, Package_TO_SOT_SMD:TO-252-2, F.Cu at (221.0, 88.0)
- U11, U12, U13, U19, U20, U21: footprint Package_SO:SO-8_3.9x4.9mm_P1.27mm -> Package_SO:SOIC-8_3.9x4.9mm_P1.27mm
- moved C22 183.7 mm to (269.6, 62.4), turned to 270 degrees
- moved U10 178.1 mm to (262.4, 59.4)
- moved TP1 169.8 mm to (275.1, 95.5)
- moved TP2 169.8 mm to (282.5, 86.6)
- moved R29 168.1 mm to (267.4, 58.6), turned to 270 degrees
- moved C19 167.9 mm to (267.4, 62.4), turned to 270 degrees
- moved C20 167.8 mm to (257.4, 59.4), turned to 270 degrees
- moved U9 164.4 mm to (248.4, 66.0), turned to 180 degrees
- moved C17 159.7 mm to (248.4, 59.8)
- moved C18 158.1 mm to (253.4, 64.4), turned to 90 degrees
- moved C16 155.8 mm to (243.4, 69.8)
- moved C15 150.5 mm to (239.8, 61.8), turned to 180 degrees
- moved U8 144.9 mm to (238.2, 65.8)
- moved R23 144.8 mm to (248.4, 62.0), turned to 180 degrees
- moved R45 142.7 mm to (243.2, 65.2), turned to 270 degrees
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- renumbered Q19 to Q18
Connections:
- Q12 pad 1: /STM32/M1_EN -> /M1/Phase_~EN
- Q13 pad 1: /STM32/M1_EN -> /M1/Phase_~EN
- Q16 pad 1: /STM32/M1_EN -> /M1/Phase_~EN
- Q17 pad 1: /STM32/M1_EN -> /M1/Phase_~EN
- Q18 pad 1: Net-(Q19-Pad1) -> Net-(Q18-Pad1)
- Q18 pad 2: /M1/phase_3/Output -> Vcc_1
- Q18 pad 3: /M1/bridge_output -> /M1/phase_3/Output
- Q27 pad 1: /STM32/M2_EN -> /M2/Phase_~EN
- Q28 pad 1: /STM32/M2_EN -> /M2/Phase_~EN
- Q31 pad 1: /STM32/M2_EN -> /M2/Phase_~EN
- Q32 pad 1: /STM32/M2_EN -> /M2/Phase_~EN
- Q35 pad 1: /STM32/M2_EN -> /M2/Phase_~EN
- Q36 pad 1: /STM32/M2_EN -> /M2/Phase_~EN
- Q8 pad 1: /STM32/M1_EN -> /M1/Phase_~EN
- Q9 pad 1: /STM32/M1_EN -> /M1/Phase_~EN
- R21 pad 1: /STM32/M1_EN -> /M1/Phase_~EN
- R60 pad 1: /STM32/M2_EN -> /M2/Phase_~EN
Routing:
- net GND: track 8.25 -> 68.3 mm, vias 0 -> 6
- net /M2/phase_1/Output: track 0.00 -> 24.6 mm
- net /M2/phase_3/Output: track 0.00 -> 24.6 mm
- net /M2/phase_2/Output: track 0.00 -> 24.6 mm
- net /M1/phase_3/Output: track 0.00 -> 24.6 mm
- net /M1/phase_1/Output: track 0.00 -> 24.6 mm
- net +3V3: track 0.00 -> 18.4 mm
- net /M2/Phase_~EN: track 0.00 -> 16.2 mm, vias 0 -> 3
- net /M1/Phase_~EN: track 0.00 -> 16.2 mm, vias 0 -> 3
- net Net-(Q27-Pad3): track 0.00 -> 13.9 mm
- net Net-(Q8-Pad3): track 0.00 -> 13.9 mm
- net Net-(Q16-Pad3): track 0.00 -> 13.9 mm
- net Net-(Q31-Pad3): track 0.00 -> 13.9 mm
- net Net-(Q35-Pad3): track 0.00 -> 13.9 mm
- net Net-(Q36-Pad3): track 0.00 -> 13.7 mm
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
Commit message: update footprints, pcb
Parts:
- added D11: D_ALT, Diode_SMD:D_2010_5025Metric_Pad1.52x2.65mm_HandSolder, F.Cu at (228.4, 51.0)
- added D12: D_ALT, Diode_SMD:D_2010_5025Metric_Pad1.52x2.65mm_HandSolder, F.Cu at (228.4, 58.4)
- added D13: D_ALT, Diode_SMD:D_2010_5025Metric_Pad1.52x2.65mm_HandSolder, F.Cu at (228.4, 65.8)
- added D14: D_ALT, Diode_SMD:D_2010_5025Metric_Pad1.52x2.65mm_HandSolder, F.Cu at (228.4, 73.2)
- added D15: D_ALT, Diode_SMD:D_2010_5025Metric_Pad1.52x2.65mm_HandSolder, F.Cu at (228.4, 80.6)
- added D16: D_ALT, Diode_SMD:D_2010_5025Metric_Pad1.52x2.65mm_HandSolder, F.Cu at (228.4, 88.0)
- added D19: D_ALT, Diode_SMD:D_2010_5025Metric_Pad1.52x2.65mm_HandSolder, F.Cu at (228.4, 95.4)
- added D20: D_ALT, Diode_SMD:D_2010_5025Metric_Pad1.52x2.65mm_HandSolder, F.Cu at (228.4, 102.8)
- added D21: D_ALT, Diode_SMD:D_2010_5025Metric_Pad1.52x2.65mm_HandSolder, F.Cu at (228.4, 110.2)
- added D22: D_ALT, Diode_SMD:D_2010_5025Metric_Pad1.52x2.65mm_HandSolder, F.Cu at (228.4, 117.6)
- added D23: D_ALT, Diode_SMD:D_2010_5025Metric_Pad1.52x2.65mm_HandSolder, F.Cu at (228.4, 125.0)
- added D24: D_ALT, Diode_SMD:D_2010_5025Metric_Pad1.52x2.65mm_HandSolder, F.Cu at (228.4, 132.4)
- added J10: M1_hall, Connector_JST:JST_XH_B5B-XH-A_1x05_P2.50mm_Vertical, F.Cu at (47.0, 122.7)
- added J11: Encoder_1, Connector_JST:JST_PH_B4B-PH-K_1x04_P2.00mm_Vertical, F.Cu at (119.3, 165.3)
- added J12: M1, Connector_Phoenix_MC:PhoenixContact_MCV_1,5_3-G-3.81_1x03_P3.81mm_Vertical, F.Cu at (47.1, 153.6)
- added J13: M1_hall, Connector_JST:JST_XH_B5B-XH-A_1x05_P2.50mm_Vertical, F.Cu at (47.0, 143.8)
- added J3: Power_1, Connector_Phoenix_MC:PhoenixContact_MCV_1,5_2-G-3.81_1x02_P3.81mm_Vertical, F.Cu at (93.4, 143.9)
- added J4: Power_2, Connector_Phoenix_MC:PhoenixContact_MCV_1,5_2-G-3.81_1x02_P3.81mm_Vertical, F.Cu at (82.3, 143.9)
- added J6: CAN_conn, Connector_JST:JST_XH_B5B-XH-A_1x05_P2.50mm_Vertical, F.Cu at (82.1, 130.5)
- added J7: CAN_conn, Connector_JST:JST_XH_B5B-XH-A_1x05_P2.50mm_Vertical, F.Cu at (82.1, 122.7)
- added J8: Encoder_1, Connector_JST:JST_PH_B4B-PH-K_1x04_P2.00mm_Vertical, F.Cu at (103.4, 165.3)
- added J9: M1, Connector_Phoenix_MC:PhoenixContact_MCV_1,5_3-G-3.81_1x03_P3.81mm_Vertical, F.Cu at (239.2, 77.0)
- added JP3: Jumper_NC_Dual, Connector_PinHeader_2.54mm:PinHeader_1x03_P2.54mm_Vertical, F.Cu at (103.2, 140.9)
- moved C22 88.1 mm to (188.2, 96.0)
- moved C19 88.1 mm to (186.0, 96.0)
- moved C20 88.1 mm to (176.0, 93.0)
- moved R29 88.1 mm to (186.0, 92.2)
- moved U10 88.1 mm to (181.0, 93.0)
- moved C15 64.1 mm to (177.6, 77.2)
- moved C16 64.1 mm to (181.2, 85.2)
- moved C17 64.1 mm to (186.2, 75.2)
- moved C18 64.1 mm to (191.2, 79.8)
- moved R23 64.1 mm to (186.2, 77.4)
- moved U9 64.1 mm to (186.2, 81.4)
- moved R45 64.1 mm to (181.0, 80.6)
- moved U8 64.1 mm to (176.0, 81.2)
- moved C56 7.67 mm to (280.1, 112.4)
- moved C57 7.67 mm to (262.2, 118.8)
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Connections:
- C48 pad 1: Net-(C48-Pad1) -> /CAN/+7V_CAN
- D10 pad 2: Net-(C48-Pad1) -> /CAN/+7V_CAN
- F3 pad 1: Net-(C48-Pad1) -> /CAN/+7V_CAN
- F3 pad 2: /CAN/+7V_CAN -> /CAN/7V_Input
- U6 pad 3: Net-(C48-Pad1) -> /CAN/+7V_CAN
Routing:
- net /M1/bridge_output: track 0.00 -> 38.0 mm
- net /M2/bridge_output: track 0.00 -> 38.0 mm
- net /M1/phase_1/Output: track 24.6 -> 51.3 mm
- net /M1/phase_3/Output: track 24.6 -> 51.1 mm
- net Vcc_1: track 0.00 -> 18.8 mm
- net Vcc_2: track 0.00 -> 18.8 mm
- net /M1/phase_2/Output: track 24.6 -> 42.8 mm
- net /M2/phase_2/Output: track 24.6 -> 35.8 mm
- net /M2/phase_1/Output: track 24.6 -> 35.8 mm
- net /M2/phase_3/Output: track 24.6 -> 35.8 mm
